File: eeprom_tagconnect.kicad_sch (KiCad schematic)
At the start: 12 parts, among them J1 Tag-Connect_TC2050-IDC-NL_2x5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, U13 TXU0304BQAR, U5 25LC512

Commit message: [#100765] Prettify decoupling caps
Parts:
- added C65: C_1u_0402, antmicro-footprints:C_0402_1005Metric, symbol antmicroCapacitors0402:C_1u_0402
Connections:
- net +1V8: now also C65.2
- net GND: now also C65.1
Other:
- moved on the sheet: C41, C43, C46, C59, J1, R27, TP26, TP27, TP28, TP29, U13, U5

Commit message: [#100765] WIP: Apply review changes
Parts:
- added R111: R_10k_0402, antmicro-footprints:R_0402_1005Metric, symbol antmicroResistors0402:R_10k_0402
- added U12: 93AA66C_SOIC, antmicro-footprints:SOIC-8_3.9x4.9x1.75mm_P1.27mm, symbol antmicroMemory:93AA66C_SOIC
Connections:
- net +3V3: now also R111.2
- net at U13.8 (OE): now also R111.1
