File: antmicro-jetson-orin-baseboard-pcie-switch-expansion-hw.kicad_pcb (KiCad board)
At the start: 0 parts

Commit message: Saved with KiCad 10
Other:
- copper layers 0 -> 2
Changed lines of the file:
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@@
 (kicad_pcb
-	(version 20241229)
-	(generator "askiff")
-	(generator_version "9.0")
+	(version 20260206)
+	(generator "pcbnew")
+	(generator_version "10.0")
+	(general
+		(thickness 1.6)
+		(legacy_teardrops no)
+	)
 	(paper "A3")
 	(title_block
@@
 		(company "Antmicro")
 	)
+	(layers
+		(0 "F.Cu" signal)
+		(2 "B.Cu" signal)
+		(9 "F.Adhes" user "F.Adhesive")
+		(11 "B.Adhes" user "B.Adhesive")
+		(13 "F.Paste" user)
+		(15 "B.Paste" user)
+		(5 "F.SilkS" user "F.Silkscreen")
+		(7 "B.SilkS" user "B.Silkscreen")
+		(1 "F.Mask" user)
+		(3 "B.Mask" user)
+		(17 "Dwgs.User" user "User.Drawings")
+		(19 "Cmts.User" user "User.Comments")
+		(21 "Eco1.User" user "User.Eco1")
+		(23 "Eco2.User" user "User.Eco2")
+		(25 "Edge.Cuts" user)
+		(27 "Margin" user)
+		(31 "F.CrtYd" user "F.Courtyard")
+		(29 "B.CrtYd" user "B.Courtyard")
+		(35 "F.Fab" user)
+		(33 "B.Fab" user)
+		(39 "User.1" user)
+		(41 "User.2" user)
+		(43 "User.3" user)
+		(45 "User.4" user)
+	)
 	(setup
-		(stackup
-			(copper_finish "ENIG")
+		(pad_to_mask_clearance 0)
+		(allow_soldermask_bridges_in_footprints no)
+		(tenting
+			(front yes)
+			(back yes)
 		)
-		(pad_to_mask_clearance 0)
+		(covering
+			(front no)
+			(back no)
+		)
+		(plugging
+			(front no)
+			(back no)
+		)
+		(capping no)
+		(filling no)
+		(pcbplotparams
+			(layerselection 0x00000000_00000000_55555555_5755f5ff)
+			(plot_on_all_layers_selection 0x00000000_00000000_00000000_00000000)
+			(disableapertmacros no)
+			(usegerberextensions no)
+			(usegerberattributes yes)
+			(usegerberadvancedattributes yes)
+			(creategerberjobfile yes)
+			(dashed_line_dash_ratio 12)
+			(dashed_line_gap_ratio 3)
+			(svgprecision 4)
+			(plotframeref no)
+			(mode 1)
+			(useauxorigin no)
+			(pdf_front_fp_property_popups yes)
+			(pdf_back_fp_property_popups yes)
+			(pdf_metadata yes)
+			(pdf_single_document no)
+			(dxfpolygonmode yes)
+			(dxfimperialunits yes)
+			(dxfusepcbnewfont yes)
+			(psnegative no)
+			(psa4output no)
+			(plot_black_and_white yes)
+			(sketchpadsonfab no)
+			(plotpadnumbers no)
+			(hidednponfab no)
+			(sketchdnponfab yes)
+			(crossoutdnponfab yes)
+			(subtractmaskfromsilk no)
+			(outputformat 1)
+			(mirror no)
+			(drillshape 1)
+			(scaleselection 1)
+			(outputdirectory "")
+		)
 	)
 	(embedded_fonts no)

Commit message: [#100645] Update stackup & prepare mock
Parts:
- added A1: Mech_M2_2242_H2.5mm, antmicro-footprints:Mech_M2_2242_H2.5mm, F.Cu at (243.9, 127.0)
- added A2: Mech_M2_2280_H2.5mm, antmicro-footprints:Mech_M2_2280_H2.5mm, F.Cu at (283.0, 100.5)
- added H1: Spacer_Drill3.7mm_H10mm_9774100151R, antmicro-footprints:Spacer_Drill3.7mm_H10mm_9774100151R, B.Cu at (194.8, 88.2)
- added H2: Spacer_Drill3.7mm_H10mm_9774100151R, antmicro-footprints:Spacer_Drill3.7mm_H10mm_9774100151R, B.Cu at (194.8, 139.7)
- added H3: Spacer_Drill3.7mm_H10mm_9774100151R, antmicro-footprints:Spacer_Drill3.7mm_H10mm_9774100151R, B.Cu at (258.9, 87.9)
- added H4: Spacer_Drill3.7mm_H10mm_9774100151R, antmicro-footprints:Spacer_Drill3.7mm_H10mm_9774100151R, B.Cu at (258.9, 139.9)
- added H5: Spacer_Drill4.4mm_H2.5mm_9774025360R, antmicro-footprints:Spacer_Drill4.4mm_H2.5mm_9774025360R, F.Cu at (243.9, 100.5)
- added H6: Spacer_Drill4.4mm_H2.5mm_9774025360R, antmicro-footprints:Spacer_Drill4.4mm_H2.5mm_9774025360R, F.Cu at (283.0, 100.5)
- added H7: Spacer_Drill4.4mm_H2.5mm_9774025360R, antmicro-footprints:Spacer_Drill4.4mm_H2.5mm_9774025360R, F.Cu at (243.9, 127.0)
- added H8: Spacer_Drill4.4mm_H2.5mm_9774025360R, antmicro-footprints:Spacer_Drill4.4mm_H2.5mm_9774025360R, F.Cu at (283.0, 127.0)
- added J1: Bus_M.2_1-2199230-6, antmicro-footprints:Bus_M.2_Socket_Key_M_TE_1-2199230-6, F.Cu at (204.1, 100.5)
- added J2: Bus_M.2_1-2199230-6, antmicro-footprints:Bus_M.2_Socket_Key_M_TE_1-2199230-6, F.Cu at (204.2, 127.2)
- added J3: OCuLink_x4_Amphenol_G14A421211112HR, antmicro-footprints:Amphenol_G14A421211112HR, B.Cu at (215.6, 87.1)
- added J4: OCuLink_x4_Amphenol_G14A421211112HR, antmicro-footprints:Amphenol_G14A421211112HR, B.Cu at (215.2, 140.9)
- added J5: OCuLink_x4_Amphenol_G14A421211112HR, antmicro-footprints:Amphenol_G14A421211112HR, B.Cu at (239.8, 140.9)
- added J6: Molex_Nano-Fit_1x2_SMD_1054301202, antmicro-footprints:Conn_Molex_Nano-Fit_1x2_SMD_1054301202, B.Cu at (243.7, 88.3)
- added J7: Plug_Samtec_ERM8_2x40_ERM8-040-05.0-L-DV-K-TR, antmicro-footprints:Conn_Plug_Samtec_ERM8_2x40_ERM8-040-05.0-L-DV-K-TR, B.Cu at (193.5, 114.7)
Routing:
- net (no net): vias 0 -> 18
Other:
- board outline added: 98.5 x 60 mm
- copper layers 2 -> 8
- board text added: "M.2 2242"
- board text added: "M.2 2280"

Commit message: [#100645] Add Antmicro and OSH logo
Parts:
- added G***: LOGO, antmicro-footprints:antmicro-logo_scaled_15mm_silk, F.Cu at (217.0, 113.1)
- added REF**: OSHW-Logo_5.7x6mm_SilkScreen, antmicro-footprints:OSHW-Logo_5.7x6mm_SilkScreen, F.Cu at (231.3, 113.8)
Other:
- board text added: "JOB PCIe Switch Expansion rev.1.0.0 07/2026"
