File: antmicro-jetson-orin-baseboard-pcie-switch-expansion-hw.kicad_pcb (KiCad board)
At the start: 8 copper layers, 98.5 x 60 mm, 338 parts, among them J1 Bus_M.2_1-2199230-6, J2 Bus_M.2_1-2199230-6, J3 OCuLink_x4_Amphenol_G14A42121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, J4 Plug_Samtec_ERM8_2x40_ERM8-04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, J5 Tag-Connect_TC2050-IDC-NL_2x5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, Q1 BSS138PW,115, Q10 BSS138PW,115, Q2 BSS138PW,115, Q3 BSS138PW,115, Q4 BSS138PW,115, Q5 BSS138PW,115, Q6 BSS138PW,115, Q7 BSS138PW,115, Q8 BSS138PW,115, Q9 BSS138PW,115, SW1 SW_CVS-02B, U10 TMUXHS4412RUAR, U11 CBTL02043ABQ, U12 TPS62A06DRLR, U13 TPS62A06DRLR, U14 SIC431AED-T1-GE3, U2 NTS0302JKZ, U4 PI7C9X3G606GP, U5 NTS0302JKZ, U6 93AA66C_SOIC, U7 SY75602BTWL-TR, U8 74LVC1G157-Q100H_SOT457, U9 NTS0302JKZ

Commit message: [#101557] Define stackup
Other:
- copper layers 8 -> 6
Changed lines of the file:
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@@
 	(generator_version "10.0")
 	(general
-		(thickness 1.62)
+		(thickness 1.73)
 		(legacy_teardrops no)
 	)
@@
 		(8 "In3.Cu" signal)
 		(10 "In4.Cu" jumper)
-		(12 "In5.Cu" signal)
-		(14 "In6.Cu" signal)
 		(2 "B.Cu" signal)
 		(9 "F.Adhes" user "F.Adhesive")
@@
 			(layer "dielectric 2"
 				(type "core")
-				(thickness 0.2)
+				(thickness 0.51)
 				(material "FR4")
 				(epsilon_r 4.39)
@@
 			(layer "dielectric 3"
 				(type "prepreg")
-				(thickness 0.12)
-				(material "PR2116")
-				(epsilon_r 4.39)
+				(thickness 0.07)
+				(material "PR1080")
+				(epsilon_r 3.91)
 				(loss_tangent 0.02) addsublayer
-				(thickness 0.12)
-				(material "PR2116")
-				(epsilon_r 4.39)
-				(loss_tangent 0)
+				(thickness 0.07)
+				(material "PR1080")
+				(epsilon_r 3.91)
+				(loss_tangent 0.02)
 			)
 			(layer "In3.Cu"
@@
 			(layer "dielectric 4"
 				(type "core")
-				(thickness 0.2)
+				(thickness 0.51)
 				(material "FR4")
 				(epsilon_r 4.39)
@@
 			(layer "dielectric 5"
 				(type "prepreg")
-				(thickness 0.12)
+				(thickness 0.1)
 				(material "PR2116")
 				(epsilon_r 4.39)
@@
 				(epsilon_r 4.39)
 				(loss_tangent 0)
-			)
-			(layer "In5.Cu"
-				(type "copper")
-				(thickness 0.035)
-			)
-			(layer "dielectric 6"
-				(type "core")
-				(thickness 0.2)
-				(material "FR4")
-				(epsilon_r 4.39)
-				(loss_tangent 0.02)
-			)
-			(layer "In6.Cu"
-				(type "copper")
-				(thickness 0.035)
-			)
-			(layer "dielectric 7"
-				(type "prepreg")
-				(thickness 0.12)
-				(material "PR2116")
-				(epsilon_r 4.3)
-				(loss_tangent 0.02)
 			)
 			(layer "B.Cu"
@@
 		(capping no)
 		(filling no)
+		(zone_defaults)
 		(pcbplotparams
 			(layerselection 0x00000000_00000000_55555555_5755f5ff)
