File: antmicro-jetson-orin-baseboard-pcie-switch-expansion-hw.kicad_pcb (KiCad board)
At the start: 6 copper layers, 98.5 x 60 mm, 343 parts, among them J1 Bus_M.2_1-2199230-6, J2 Bus_M.2_1-2199230-6, J3 OCuLink_x4_Amphenol_G14A42121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, J4 Plug_Samtec_ERM8_2x40_ERM8-04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, J5 Tag-Connect_TC2050-IDC-NL_2x5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, Q1 BSS138PW,115, Q10 BSS138PW,115, Q2 BSS138PW,115, Q3 BSS138PW,115, Q4 BSS138PW,115, Q5 BSS138PW,115, Q6 BSS138PW,115, Q7 BSS138PW,115, Q8 BSS138PW,115, Q9 BSS138PW,115, SW1 SW_CVS-02B, U10 TMUXHS4412RUAR, U11 CBTL02043ABQ, U12 TPS62A06DRLR, U13 TPS62A06DRLR, U14 SIC431AED-T1-GE3, U2 NTS0302JKZ, U4 PI7C9X3G606GP, U5 NTS0302JKZ, U6 93AA66C_SOIC, U7 SY75602BTWL-TR, U8 74LVC1G157-Q100H_SOT457, U9 NTS0302JKZ

Commit message: [#102081] Place 0V95 decoupling caps
Parts:
- moved C40 108.2 mm to (220.8, 115.7), turned to 180 degrees
- moved C38 103.4 mm to (220.8, 114.8), turned to 0 degrees
- moved C34 101.0 mm to (219.8, 113.8)
- moved C30 100.8 mm to (216.7, 113.4), turned to 180 degrees
- moved C45 100.6 mm to (221.2, 113.5), turned to 90 degrees
- moved C51 99.2 mm to (216.7, 112.5), turned to 0 degrees
- moved C39 99.1 mm to (219.4, 115.3), turned to 90 degrees
- moved C52 97.9 mm to (216.7, 111.5)
- moved C33 97.6 mm to (216.7, 114.4), turned to 180 degrees
- moved C37 97.3 mm to (218.4, 113.5), turned to 90 degrees
- moved C35 96.8 mm to (218.4, 115.3), turned to -90 degrees
- moved C50 95.0 mm to (219.8, 112.4), turned to 180 degrees
Routing:
- net +0V95: track 7.35 -> 8.15 mm, vias 10 -> 12
