File: supply.kicad_sch (KiCad schematic)
At the start: 60 parts, among them Q1 BSS138PW,115, Q6 BSS138PW,115, U21 TPS62A06DRLR, U22 TPS62A06DRLR, U40 SIC431AED-T1-GE3

Commit message: [#100765] Apply fixes from review
Parts:
- added TP33, TP41: TP_0.75mm_SMD, antmicro-footprints:TP_SMD_0.75mm, symbol antmicroTestPoints:TP_0.75mm_SMD
Connections:
- net at R71.2, U21.6 (PG): now also TP33.1
- net at R79.2, U22.6 (PG): now also TP41.1
Other:
- note removed: "TODO: add TVS"
