File: supply.kicad_sch (KiCad schematic)
At the start: 62 parts, among them Q10 BSS138PW,115, Q9 BSS138PW,115, U12 TPS62A06DRLR, U13 TPS62A06DRLR, U14 SIC431AED-T1-GE3

Commit message: [#101557] Routing
Parts:
- removed D10, D11: LED_G_0603_LG_L29K-G2J1-24-Z, antmicro-footprints:LED_0603_1608Metric_G, symbol antmicroLEDIndicationDiscrete:LED_G_0603_LG_L29K-G2J1-24-Z
- removed TP46, TP47, TP48, TP49, TP50: TP_0.75mm_SMD, antmicro-footprints:TP_SMD_0.75mm, symbol antmicroTestPoints:TP_0.75mm_SMD
- added D10, D11: LED_G_0603_KP-1608CGCK, antmicro-footprints:LED_0603_1608Metric_G, symbol antmicroLEDIndicationDiscrete:LED_G_0603_KP-1608CGCK
- added TP46, TP47, TP48, TP49, TP50, TP53, TP54, TP55: TP_1mm_SMD, antmicro-footprints:TP_SMD_1mm, symbol antmicroTestPoints:TP_1mm_SMD
Connections:
- net +0V95: now also TP48.1, TP53.1
- net +1V8: now also TP49.1, TP54.1
- net +3V3: now also TP50.1, TP55.1
- net at R118.1: now also D11.2 (A)
- net at R117.1: now also D10.2 (A)
- net at Q10.3 (D): now also D11.1 (C)
- net at R125.2, U12.6 (PG): now also TP46.1
- net at R126.2, U13.6 (PG): now also TP47.1
- net at Q9.3 (D): now also D10.1 (C)

Commit message: [#105687] Rename project, mention img in README
Other:
- title: antmicro-jetson-orin-baseboard-pcie-switch-expansion-hw -> jetson-orin-baseboard-pcie-switch-expansion
