File: expansion-conn.kicad_sch (KiCad schematic)
At the start: 15 parts, among them J7 Plug_Samtec_ERM8_2x40_ERM8-04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

Commit message: [#100765] Reset designators
Parts:
- renumbered C57 to C22, C56 to C23, J7 to J4, R117 to R30, R118 to R31, TP4 to TP10, TP42 to TP11, TP43 to TP12, TP2 to TP13, TP18 to TP14, TP19 to TP15, TP20 to TP16, TP21 to TP17, TP22 to TP18, TP23 to TP9
Changed lines of the file:
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@@
 		(dnp no)
 		(fields_autoplaced yes)
-		(property "Reference" "C57"
+		(property "Reference" "C22"
 			(at 168.91 199.3836 90)
 			(show_name no)
@@
 			(project "antmicro-jetson-orin-baseboard-pcie-switch-expansion-hw"
 				(path "/9f8272ef-d62d-4578-9094-a2852fcd4bf4/e2953c32-de4d-49db-967a-cd128c95e407"
-					(reference "C57")
+					(reference "C22")
 					(unit 1)
 				)
@@
 		(in_pos_files yes)
 		(dnp no)
-		(property "Reference" "#PWR02"
+		(property "Reference" "#PWR045"
 			(at 175.26 186.69 0)
 			(hide yes)
@@
 			(project "antmicro-jetson-orin-baseboard-pcie-switch-expansion-hw"
 				(path "/9f8272ef-d62d-4578-9094-a2852fcd4bf4/e2953c32-de4d-49db-967a-cd128c95e407"
-					(reference "#PWR02")
+					(reference "#PWR045")
 					(unit 1)
 				)
@@
 		(in_pos_files yes)
 		(dnp no)
-		(property "Reference" "#PWR09"
+		(property "Reference" "#PWR048"
 			(at 229.87 186.69 0)
 			(hide yes)
@@
 			(project "antmicro-jetson-orin-baseboard-pcie-switch-expansion-hw"
 				(path "/9f8272ef-d62d-4578-9094-a2852fcd4bf4/e2953c32-de4d-49db-967a-cd128c95e407"
-					(reference "#PWR09")
+					(reference "#PWR048")
 					(unit 1)
 				)
@@
 		(dnp no)
 		(fields_autoplaced yes)
-		(property "Reference" "#PWR04"
+		(property "Reference" "#PWR047"
 			(at 218.44 199.39 0)
 			(hide yes)
@@
 			(project "antmicro-jetson-orin-baseboard-pcie-switch-expansion-hw"
 				(path "/9f8272ef-d62d-4578-9094-a2852fcd4bf4/e2953c32-de4d-49db-967a-cd128c95e407"
-					(reference "#PWR04")
+					(reference "#PWR047")
 					(unit 1)
 				)
@@
 		(dnp yes)
 		(fields_autoplaced yes)
-		(property "Reference" "C56"
+		(property "Reference" "C23"
 			(at 177.8 175.2536 90)
 			(show_name no)
@@
 			(project "antmicro-jetson-orin-baseboard-pcie-switch-expansion-hw"
 				(path "/9f8272ef-d62d-4578-9094-a2852fcd4bf4/e2953c32-de4d-49db-967a-cd128c95e407"
-					(reference "C56")
+					(reference "C23")
 					(unit 1)
 				)
@@
 		(in_pos_files yes)
 		(dnp no)
-		(property "Reference" "TP20"
+		(property "Reference" "TP16"
 			(at 192.786 153.67 0)
 			(show_name no)
@@
 			(project "antmicro-jetson-orin-baseboard-pcie-switch-expansion-hw"
 				(path "/9f8272ef-d62d-4578-9094-a2852fcd4bf4/e2953c32-de4d-49db-967a-cd128c95e407"
-					(reference "TP20")
+					(reference "TP16")
 					(unit 1)
 				)
@@
 		(dnp no)
 		(fields_autoplaced yes)
-		(property "Reference" "#FLG010"
+		(property "Reference" "#FLG03"
 			(at 155.575 195.58 0)
 			(hide yes)
@@
 			(project "antmicro-jetson-orin-baseboard-pcie-switch-expansion-hw"
 				(path "/9f8272ef-d62d-4578-9094-a2852fcd4bf4/e2953c32-de4d-49db-967a-cd128c95e407"
-					(reference "#FLG010")
+					(reference "#FLG03")
 					(unit 1)
 				)
@@
 		(dnp no)
 		(fields_autoplaced yes)
-		(property "Reference" "J7"
+		(property "Reference" "J4"
 			(at 208.915 77.47 0)
 			(show_name no)
@@
 			(project "antmicro-jetson-orin-baseboard-pcie-switch-expansion-hw"
 				(path "/9f8272ef-d62d-4578-9094-a2852fcd4bf4/e2953c32-de4d-49db-967a-cd128c95e407"
-					(reference "J7")
+					(reference "J4")
 					(unit 1)
 				)
@@
 		(in_pos_files yes)
 		(dnp no)
-		(property "Reference" "TP43"
+		(property "Reference" "TP12"
 			(at 181.356 170.18 0)
 			(show_name no)
@@
 			(project "antmicro-jetson-orin-baseboard-pcie-switch-expansion-hw"
 				(path "/9f8272ef-d62d-4578-9094-a2852fcd4bf4/e2953c32-de4d-49db-967a-cd128c95e407"
-					(reference "TP43")
+					(reference "TP12")
 					(unit 1)
 				)
@@
 		(in_pos_files yes)
 		(dnp no)
-		(property "Reference" "#PWR053"
+		(property "Reference" "#PWR044"
 			(at 166.37 210.82 0)
 			(hide yes)
@@
 			(project "antmicro-jetson-orin-baseboard-pcie-switch-expansion-hw"
 				(path "/9f8272ef-d62d-4578-9094-a2852fcd4bf4/e2953c32-de4d-49db-967a-cd128c95e407"
-					(reference "#PWR053")
+					(reference "#PWR044")
 					(unit 1)
 				)
@@
 		(dnp no)
 		(fields_autoplaced yes)
-		(property "Reference" "#PWR03"
+		(property "Reference" "#PWR046"
 			(at 199.39 199.39 0)
 			(hide yes)
@@
 			(project "antmicro-jetson-orin-baseboard-pcie-switch-expansion-hw"
 				(path "/9f8272ef-d62d-4578-9094-a2852fcd4bf4/e2953c32-de4d-49db-967a-cd128c95e407"
-					(reference "#PWR03")
+					(reference "#PWR046")
 					(unit 1)
 				)
@@
 		(in_pos_files yes)
 		(dnp no)
-		(property "Reference" "TP21"
+		(property "Reference" "TP17"
 			(at 192.786 156.21 0)
 			(show_name no)
@@
 			(project "antmicro-jetson-orin-baseboard-pcie-switch-expansion-hw"
 				(path "/9f8272ef-d62d-4578-9094-a2852fcd4bf4/e2953c32-de4d-49db-967a-cd128c95e407"
-					(reference "TP21")
+					(reference "TP17")
 					(unit 1)
 				)
@@
 		(in_pos_files yes)
 		(dnp no)
-		(property "Reference" "TP22"
+		(property "Reference" "TP18"
 			(at 192.786 158.75 0)
 			(show_name no)
@@
 			(project "antmicro-jetson-orin-baseboard-pcie-switch-expansion-hw"
 				(path "/9f8272ef-d62d-4578-9094-a2852fcd4bf4/e2953c32-de4d-49db-967a-cd128c95e407"
-					(reference "TP22")
+					(reference "TP18")
 					(unit 1)
 				)
@@
 		(dnp no)
 		(fields_autoplaced yes)
-		(property "Reference" "#FLG01"
+		(property "Reference" "#FLG05"
 			(at 242.57 201.295 0)
 			(hide yes)
@@
 			(project "antmicro-jetson-orin-baseboard-pcie-switch-expansion-hw"
 				(path "/9f8272ef-d62d-4578-9094-a2852fcd4bf4/e2953c32-de4d-49db-967a-cd128c95e407"
-					(reference "#FLG01")
+					(reference "#FLG05")
 					(unit 1)
 				)
@@
 		(in_pos_files yes)
 		(dnp no)
-		(property "Reference" "R117"
+		(property "Reference" "R30"
 			(at 165.1 121.412 0)
 			(show_name no)
@@
 			(project "antmicro-jetson-orin-baseboard-pcie-switch-expansion-hw"
 				(path "/9f8272ef-d62d-4578-9094-a2852fcd4bf4/e2953c32-de4d-49db-967a-cd128c95e407"
-					(reference "R117")
+					(reference "R30")
 					(unit 1)
 				)
@@
 		(dnp no)
 		(fields_autoplaced yes)
-		(property "Reference" "TP4"
+		(property "Reference" "TP10"
 			(at 177.8 189.865 90)
 			(show_name no)
@@
 			(project "antmicro-jetson-orin-baseboard-pcie-switch-expansion-hw"
 				(path "/9f8272ef-d62d-4578-9094-a2852fcd4bf4/e2953c32-de4d-49db-967a-cd128c95e407"
-					(reference "TP4")
+					(reference "TP10")
 					(unit 1)
 				)
@@
 		(in_pos_files yes)
 		(dnp no)
-		(property "Reference" "#PWR044"
+		(property "Reference" "#PWR043"
 			(at 160.02 195.58 0)
 			(hide yes)
@@
 			(project "antmicro-jetson-orin-baseboard-pcie-switch-expansion-hw"
 				(path "/9f8272ef-d62d-4578-9094-a2852fcd4bf4/e2953c32-de4d-49db-967a-cd128c95e407"
-					(reference "#PWR044")
+					(reference "#PWR043")
 					(unit 1)
 				)
@@
 		(dnp no)
 		(fields_autoplaced yes)
-		(property "Reference" "#FLG011"
+		(property "Reference" "#FLG04"
 			(at 235.585 184.15 0)
 			(hide yes)
@@
 			(project "antmicro-jetson-orin-baseboard-pcie-switch-expansion-hw"
 				(path "/9f8272ef-d62d-4578-9094-a2852fcd4bf4/e2953c32-de4d-49db-967a-cd128c95e407"
-					(reference "#FLG011")
+					(reference "#FLG04")
 					(unit 1)
 				)
@@
 		(in_pos_files yes)
 		(dnp no)
-		(property "Reference" "TP19"
+		(property "Reference" "TP15"
 			(at 192.786 151.13 0)
 			(show_name no)
@@
 			(project "antmicro-jetson-orin-baseboard-pcie-switch-expansion-hw"
 				(path "/9f8272ef-d62d-4578-9094-a2852fcd4bf4/e2953c32-de4d-49db-967a-cd128c95e407"
-					(reference "TP19")
+					(reference "TP15")
 					(unit 1)
 				)
@@
 		(in_pos_files yes)
 		(dnp no)
-		(property "Reference" "TP2"
+		(property "Reference" "TP13"
 			(at 189.23 191.77 0)
 			(show_name no)
@@
 			(project "antmicro-jetson-orin-baseboard-pcie-switch-expansion-hw"
 				(path "/9f8272ef-d62d-4578-9094-a2852fcd4bf4/e2953c32-de4d-49db-967a-cd128c95e407"
-					(reference "TP2")
+					(reference "TP13")
 					(unit 1)
 				)
@@
 		(in_pos_files yes)
 		(dnp no)
-		(property "Reference" "TP42"
+		(property "Reference" "TP11"
 			(at 181.356 167.64 0)
 			(show_name no)
@@
 			(project "antmicro-jetson-orin-baseboard-pcie-switch-expansion-hw"
 				(path "/9f8272ef-d62d-4578-9094-a2852fcd4bf4/e2953c32-de4d-49db-967a-cd128c95e407"
-					(reference "TP42")
+					(reference "TP11")
 					(unit 1)
 				)
@@
 		(in_pos_files yes)
 		(dnp no)
-		(property "Reference" "R118"
+		(property "Reference" "R31"
 			(at 165.1 130.556 0)
 			(show_name no)
@@
 			(project "antmicro-jetson-orin-baseboard-pcie-switch-expansion-hw"
 				(path "/9f8272ef-d62d-4578-9094-a2852fcd4bf4/e2953c32-de4d-49db-967a-cd128c95e407"
-					(reference "R118")
+					(reference "R31")
 					(unit 1)
 				)
@@
 		(in_pos_files yes)
 		(dnp no)
-		(property "Reference" "TP18"
+		(property "Reference" "TP14"
 			(at 192.786 148.59 0)
 			(show_name no)
@@
 			(project "antmicro-jetson-orin-baseboard-pcie-switch-expansion-hw"
 				(path "/9f8272ef-d62d-4578-9094-a2852fcd4bf4/e2953c32-de4d-49db-967a-cd128c95e407"
-					(reference "TP18")
+					(reference "TP14")
 					(unit 1)
 				)
@@
 		(in_pos_files yes)
 		(dnp no)
-		(property "Reference" "TP23"
+		(property "Reference" "TP9"
 			(at 171.196 171.45 0)
 			(show_name no)
@@
 			(project "antmicro-jetson-orin-baseboard-pcie-switch-expansion-hw"
 				(path "/9f8272ef-d62d-4578-9094-a2852fcd4bf4/e2953c32-de4d-49db-967a-cd128c95e407"
-					(reference "TP23")
+					(reference "TP9")
 					(unit 1)
 				)
