File: oculink.kicad_sch (KiCad schematic)
At the start: 28 parts, among them J3 OCuLink_x4_Amphenol_G14A42121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, U2 NTS0302JKZ

Commit message: [#101557] Routing
Connections:
- net +3V3: no longer U1.4 (EN)
- net +5V: no longer U3.4 (EN)
- new net ~{PCIE_{MUX_CH}}: U1.4 (EN), U3.4 (EN)
Changed lines of the file:
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@@
 	(title_block
 		(title "antmicro-jetson-orin-baseboard-pcie-switch-expansion-hw")
-		(date "2026-08-11")
+		(date "2026-08-26")
 		(rev "1.0.0")
 		(company "Antmicro")
@@
 	)
 	(junction
-		(at 160.02 191.77)
-		(diameter 0)
-		(color 0 0 0 0)
-	)
-	(junction
 		(at 99.06 119.38)
 		(diameter 0)
@@
 	)
 	(junction
-		(at 71.12 191.77)
-		(diameter 0)
-		(color 0 0 0 0)
-	)
-	(junction
 		(at 127 100.33)
 		(diameter 0)
@@
 	(wire
 		(pts
-			(xy 160.02 196.85) (xy 162.56 196.85)
+			(xy 293.37 190.5) (xy 330.2 190.5)
 		)
 		(stroke
@@
 	(wire
 		(pts
-			(xy 293.37 190.5) (xy 330.2 190.5)
+			(xy 293.37 160.02) (xy 330.2 160.02)
 		)
 		(stroke
@@
 	(wire
 		(pts
-			(xy 293.37 160.02) (xy 330.2 160.02)
+			(xy 63.5 186.69) (xy 71.12 186.69)
 		)
 		(stroke
@@
 	(wire
 		(pts
-			(xy 63.5 186.69) (xy 71.12 186.69)
+			(xy 72.39 196.85) (xy 73.66 196.85)
 		)
 		(stroke
@@
 	(wire
 		(pts
-			(xy 71.12 196.85) (xy 73.66 196.85)
-		)
-		(stroke
-			(width 0)
-			(type default)
-		)
-	)
-	(wire
-		(pts
 			(xy 95.25 200.66) (xy 95.25 201.93)
 		)
@@
 	(wire
 		(pts
+			(xy 161.29 196.85) (xy 162.56 196.85)
+		)
+		(stroke
+			(width 0)
+			(type default)
+		)
+	)
+	(wire
+		(pts
 			(xy 152.4 186.69) (xy 152.4 187.96)
 		)
@@
 	(wire
 		(pts
-			(xy 160.02 191.77) (xy 160.02 196.85)
-		)
-		(stroke
-			(width 0)
-			(type default)
-		)
-	)
-	(wire
-		(pts
 			(xy 104.14 119.38) (xy 99.06 119.38)
 		)
@@
 	(wire
 		(pts
-			(xy 71.12 191.77) (xy 71.12 196.85)
-		)
-		(stroke
-			(width 0)
-			(type default)
-		)
-	)
-	(wire
-		(pts
 			(xy 99.06 125.73) (xy 99.06 127)
 		)
@@
 		)
 	)
+	(global_label "~{PCIE_{MUX_CH}}"
+		(shape input)
+		(at 161.29 196.85 180)
+		(fields_autoplaced yes)
+		(effects
+			(font
+				(size 1.27 1.27)
+			)
+			(justify right)
+		)
+		(property "Intersheetrefs" "${INTERSHEET_REFS}"
+			(at 147.9126 196.85 0)
+			(hide yes)
+			(show_name no)
+			(do_not_autoplace no)
+			(effects
+				(font
+					(size 1.27 1.27)
+				)
+				(justify right)
+			)
+		)
+	)
+	(global_label "~{PCIE_{MUX_CH}}"
+		(shape input)
+		(at 72.39 196.85 180)
+		(fields_autoplaced yes)
+		(effects
+			(font
+				(size 1.27 1.27)
+			)
+			(justify right)
+		)
+		(property "Intersheetrefs" "${INTERSHEET_REFS}"
+			(at 59.0126 196.85 0)
+			(hide yes)
+			(show_name no)
+			(do_not_autoplace no)
+			(effects
+				(font
+					(size 1.27 1.27)
+				)
+				(justify right)
+			)
+		)
+	)

Commit message: [#105687] Rename project, mention img in README
Other:
- title: antmicro-jetson-orin-baseboard-pcie-switch-expansion-hw -> jetson-orin-baseboard-pcie-switch-expansion
