File: pcie-mux.kicad_sch (KiCad schematic)
At the start: 51 parts, among them Q6 BSS138PW,115, Q7 BSS138PW,115, Q8 BSS138PW,115, SW1 SW_CVS-02B, U10 TMUXHS4412RUAR, U11 CBTL02043ABQ, U7 SY75602BTWL-TR, U8 74LVC1G157-Q100H_SOT457, U9 NTS0302JKZ

Commit message: [#101557] Routing
Parts:
- removed D8, D9: LED_G_0603_LG_L29K-G2J1-24-Z, antmicro-footprints:LED_0603_1608Metric_G, symbol antmicroLEDIndicationDiscrete:LED_G_0603_LG_L29K-G2J1-24-Z
- added D8, D9: LED_G_0603_KP-1608CGCK, antmicro-footprints:LED_0603_1608Metric_G, symbol antmicroLEDIndicationDiscrete:LED_G_0603_KP-1608CGCK
Connections:
- net +3V3: now also D8.2 (A), D9.2 (A)
- net ~{PCIE_{MUX_CH}}: now reaches Q6.3 (D), Q8.1 (G), R84.1, R86.1
- net at R84.2: now also D8.1 (C)
- net at R88.2: now also D9.1 (C)
Other:
- moved on the sheet: R95

Commit message: [#105687] Rename project, mention img in README
Other:
- title: antmicro-jetson-orin-baseboard-pcie-switch-expansion-hw -> jetson-orin-baseboard-pcie-switch-expansion
